File: pcbs/corne-cherry/hotswap/corne-cherry.kicad_sch (KiCad schematic)
At the start: 0 parts

Commit message: fixes and preparing for pcba
Other:
- company: foostan -> tomislavrekic
Changed lines of the file:
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@@
 	(title_block
 		(title "Corne")
-		(date "2024-05-07")
-		(rev "4.1.0")
-		(company "foostan")
+		(date "2025-01-21")
+		(rev "4.1.0-USB")
+		(company "tomislavrekic")
 	)
 	(sheet
